File: EAGLE/untitled.brd (EAGLE design)
At the start: 86.2 x 53.6 mm, 56 parts, among them IC1 MIC29302WU, IC3 FT231XS-R, IC6 SMF05CT2G, J13 693023010811, Q1 MMBT3904, U6 SI2301BDS-T1-E3

Commit message: FEAT: update route pcb
Parts:
- added JP1, JP2: (no value), pinhead:1X03
- moved PSU_EN 15.7 mm to (9.40, 46.5), turned to 90 degrees
- moved R6 4.59 mm to (10.4, 41.8)
- moved R5 4.58 mm to (11.9, 41.8)
- moved Q1 0.85 mm to (15.5, 38.0)
- moved R14 0.13 mm to (14.6, 9.78), turned to 180 degrees
- moved SERIALMCU 0.13 mm to (2.79, 37.8)
- turned R15 to 180 degrees
Connections:
- new net D+_IC: IC3.11, JP1.1
- new net D+_USB: JP1.3, USB.A6, USB.B6
- new net D-_IC: IC3.12, JP2.1
- new net D-_USB: JP2.3, USB.A7, USB.B7
- net D+: now also JP1.2; no longer USB.A6, USB.B6
- net D-: now also JP2.2; no longer USB.A7, USB.B7
Routing:
- net EC20_3V3: track 0.00 -> 120.1 mm, vias 0 -> 2
- net D-_IC: track 0.00 -> 86.7 mm, vias 0 -> 1
- net D+_IC: track 0.00 -> 76.6 mm, vias 0 -> 1
- net TXD: track 0.00 -> 74.6 mm, vias 0 -> 2
- net RXD: track 0.00 -> 69.6 mm, vias 0 -> 2
- net EC20_LED_WWAN: track 0.00 -> 61.5 mm, vias 0 -> 4
- net +5V: track 0.00 -> 57.1 mm
- net EC20_RST: track 0.00 -> 54.5 mm, vias 0 -> 2
- net EC20_SIM_VCC: track 0.00 -> 48.8 mm, vias 0 -> 5
- net EC20_SIM_CLK: track 0.00 -> 47.6 mm, vias 0 -> 3
- net EC20_WAKEUP: track 0.00 -> 47.0 mm, vias 0 -> 3
- net EC20_SIM_DATA: track 0.00 -> 39.6 mm, vias 0 -> 3
- net D+_USB: track 0.00 -> 36.4 mm, vias 0 -> 2
- net EC20_SIM_RST: track 0.00 -> 33.8 mm, vias 0 -> 3
- net D-_USB: track 0.00 -> 33.1 mm, vias 0 -> 2
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- added copper zone on layer 1, net GND
- added copper zone on layer 16, net GND
Other:
- board text added: "MINI PCIE TO UART USB"
- board text added: "POSITRON ELEKTRONIK"
