File: EAGLE/mini_pcie_to_uart_usb.sch (EAGLE design)
At the start: 54 parts, among them IC1 MIC29302WU, IC3 FT231XS-R, IC6 SMF05CT2G, J13 693023010811, Q1 MMBT3904, U6 SI2301BDS-T1-E3

Commit message: FEAT: update 3d pcb
Parts:
- added H5, H6: 3MM_HOLE, 3mm_special_hole:3MM_HOLE
- added JP1, JP2: (no value), pinhead:PINHD-1X3
Connections:
- new net D+_IC: IC3.USBDP, JP1.1
- new net D+_USB: JP1.3, USB.DP1, USB.DP2
- new net D-_IC: IC3.USBDM, JP2.1
- new net D-_USB: JP2.3, USB.DN1, USB.DN2
- net D+: now also JP1.2; no longer USB.DP1, USB.DP2
- net D-: now also JP2.2; no longer USB.DN1, USB.DN2
