File: EAGLE/mini_pcie_to_uart_usb.brd (EAGLE design)
At the start: 86.2 x 53.6 mm, 58 parts, among them IC1 MIC29302WU, IC3 FT231XS-R, IC6 SMF05CT2G, J13 693023010811, Q1 MMBT3904, U6 SI2301BDS-T1-E3

Commit message: FEAT: update pcb and file documentation
Parts:
- moved H1 5.15 mm to (70.3, 30.9)
- moved H3 5.11 mm to (70.3, 6.96)
- moved MODEM 0.18 mm to (22.4, 19.1), turned to 270 degrees
Routing:
- net EC20_3V3: track 120.1 -> 182.9 mm
- net N$41: track 3.13 -> 24.1 mm, vias 0 -> 2
- net N$40: track 3.37 -> 23.5 mm, vias 0 -> 2
- net EC20_SIM_VCC: track 48.8 -> 57.7 mm
- net EC20_WAKEUP: track 47.0 -> 54.4 mm
- net EC20_LED_WWAN: track 61.5 -> 68.0 mm, vias 4 -> 2
- net EC20_SIM_RST: track 33.8 -> 39.2 mm
- net EC20_SIM_CLK: track 47.6 -> 42.7 mm
- net EC20_SIM_DATA: track 39.6 -> 35.2 mm, vias 3 -> 1
- net EC20_RST: track 54.5 -> 51.0 mm
